File: hardware/VCO-Simple-Back.brd (EAGLE design)
At the start: 29.2 x 97.8 mm, 85 parts, among them IC1 TL071, IC2 V3340SO16, IC3 LM397, IC4 TL072, IC5 TL072, P1 POWER_SIMPLE10_SHROUDED, Q1 3904, Q2 3904, U1 LM79L05A, U2 MC78L05A

Commit message: revised component values
Parts:
- DRIVE, R24: value 10K -> 100K
- R14: value 100K -> 200K
- R27: value 100K -> 10K
- R32: value 10K -> 1K
- R6: value 100K -> 150K
